Commit message: Fixed URDF file

File: data/planar2R.urdf (robot description, URDF)
Before this commit: robot Planar 2R robot, 4 links, 3 joints
Joints:
- joint end_effector: child (none) -> end_effector; parent (none) -> link_2
- joint joint_1: limit (none) -> lower=-3.141593 upper=3.141593 effort=100 velocity=3.1415926; origin xyz=1 0 0 rpy=0 0 0 -> xyz=0 0 0 rpy=0 0 0
- joint joint_2: limit (none) -> lower=-3.141593 upper=3.141593 effort=100 velocity=3.1415926

Commit message: Updated for Klamp't 0.8 structure

File: data/planar2R.urdf (robot description, URDF)
Before this commit: robot Planar 2R robot, 4 links, 3 joints
Joints:
- joint end_effector: origin xyz=2 0 0 -> xyz=1 0 0
